File: pcb/psu.kicad_sch (KiCad schematic)
At the start: 0 parts

Commit message: Updating schematic based on review from Mike
Parts:
- added C10, C4, C5, C8: DNP, Capacitor_SMD:C_1206_3216Metric_Pad1.33x1.80mm_HandSolder, symbol Device:C
- added C3, C6: 10u, Capacitor_SMD:C_1206_3216Metric_Pad1.33x1.80mm_HandSolder, symbol Device:C
- added C7, C9: 22u, Capacitor_SMD:C_1206_3216Metric_Pad1.33x1.80mm_HandSolder, symbol Device:C
- added D1, D2: LED, LED_SMD:LED_0603_1608Metric_Pad1.05x0.95mm_HandSolder, symbol Device:LED
- added R2, R3, R4, R5: DNP, Resistor_SMD:R_0603_1608Metric_Pad0.98x0.95mm_HandSolder, symbol Device:R
- added R6: 1K, Resistor_SMD:R_0603_1608Metric_Pad0.98x0.95mm_HandSolder, symbol Device:R
- added R7: 2.7K, Resistor_SMD:R_0603_1608Metric_Pad0.98x0.95mm_HandSolder, symbol Device:R
- added U4: K78L05-3AR3, dmxaudio:K78LXX-3AR3, symbol dmxaudio:K78L05-3AR3
- added U5: K78L12-3AR3, dmxaudio:K78LXX-3AR3, symbol dmxaudio:K78L12-3AR3
Connections:
- new net: D2.2 (A), R7.2
- new net: D1.2 (A), R6.2
- new net: R4.1, R5.2, U5.12 (TRIM)
- new net: R2.1, R3.2, U4.12 (TRIM)
- new net +12V: C10.1, C9.1, R5.1, R7.1, U5.10 (+VO), U5.11 (+V0), U5.9 (+VO)
- new net +24V: C3.1, C4.1, C5.1, C6.1, U4.2 (VIN), U4.3 (VIN), U4.4 (VIN), U5.2 (VIN), U5.3 (VIN), U5.4 (VIN)
- new net +5V: C7.1, C8.1, R3.1, R6.1, U4.10 (+VO), U4.11 (+V0), U4.9 (+VO)
- new net GND: C10.2, C3.2, C4.2, C5.2, C6.2, C7.2, C8.2, C9.2, D1.1 (K), D2.1 (K), R2.2, R4.2, U4.5 (GND), U4.6 (GND), U4.7 (GND), U4.8 (GND), U5.5 (GND), U5.6 (GND), U5.7 (GND), U5.8 (GND)
- no-connect marks 0 -> 2
