File: pcb/amplifier.kicad_sch (KiCad schematic)
At the start: 0 parts

Commit message: Updating schematic based on review from Mike
Parts:
- added C11: 470u DNP, symbol Device:C_Polarized_Small
- added C7 (x2): 22u DNP, Capacitor_SMD:C_1206_3216Metric_Pad1.33x1.80mm_HandSolder, symbol Device:C
- added R3 (x2): DNP, Resistor_SMD:R_0603_1608Metric_Pad0.98x0.95mm_HandSolder, symbol Device:R
- added U6: CJMCU-8006, dmxaudio:CJMCU-8006, symbol dmxaudio:CJMCU-8006
Connections:
- new net 12V: C11.1, C7.1, U6.10 (PVCCR), U6.11 (PVCCL), U6.9 (AVCC)
- new net 5V: C7.1, R3.1, U6.13 (AVDD), U6.14 (AVDD)
- new net GND: C11.2, C7.2, C7.2, R3.2, U6.12 (GND), U6.16 (GND), U6.2 (GND), U6.3 (LINP), U6.4 (RINP), U6.5 (GND), U6.7 (GND)
- new net LEFT: U6.1 (LINN)
- new net MUTE: R3.1, U6.15 (MUTE)
- new net RIGHT: U6.6 (RINN)
- new net SPEAKER_L+: U6.18 (LP+)
- new net SPEAKER_L-: U6.17 (LN-)
- new net SPEAKER_R+: U6.20 (RP+)
- new net SPEAKER_R-: U6.19 (RN-)
- new net ~{SD}: R3.2, U6.8 (~{SD})
Other:
- note added: "PAM8006A data sheet says ground INP for single-ended input"
- note added: "SD and MUTE have V_ih_min = 2.0V, so will work with 3.3V outputs"

Commit message: Adding PCB files sent off to fab
Parts:
- C11: footprint (none) -> Capacitor_THT:CP_Radial_D8.0mm_P2.50mm
Changed lines of the file:
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@@
       (effects (font (size 1.27 1.27)) (justify left))
     )
-    (property "Footprint" "" (at 177.8 76.2 0)
+    (property "Footprint" "Capacitor_THT:CP_Radial_D8.0mm_P2.50mm" (at 177.8 76.2 0)
       (effects (font (size 1.27 1.27)) hide)
     )
