File: pcb/dmxaudio.kicad_sch (KiCad schematic)
At the start: 12 parts, among them J1 USB_A, J2 RJ45, J3 RJ45_Bel_SI-60062-F, J4 Conn_01x04, J5 Conn_01x03, J6 Conn_01x04

Commit message: Adding PCB files sent off to fab
Parts:
- added Brd1: SSD1306, dmxaudio:128x64OLED, symbol SSD1306-128x64_OLED:SSD1306
- added J7: Conn_01x06, Connector_Molex:Molex_KK-254_AE-6410-06A_1x06_P2.54mm_Vertical, symbol Connector_Generic:Conn_01x06
- F1: footprint Fuse:Fuseholder_Clip-5x20mm_Keystone_3517_Inline_P23.11x6.76mm_D1.70mm_Horizontal -> dmxaudio:XF-506P
Connections:
- net +3V3: now also Brd1.2 (VCC)
- net GND: now also Brd1.1 (GND), J7.1 (Pin_1), J7.2 (Pin_2)
- net MCU/RS485_A: now also J7.6 (Pin_6)
- net MCU/RS485_B: now also J7.5 (Pin_5)
- net MCU/SCL: now also Brd1.3 (SCL)
- net MCU/SDA: now also Brd1.4 (SDA)
- net 24V_PREFUSE: now reaches F1.1, J2.4, J2.5
- net 24V_PREFUSE: now also J7.3 (Pin_3), J7.4 (Pin_4)
Changed lines of the file:
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@@
   (junction (at 165.1 148.59) (diameter 0) (color 0 0 0 0)
   )
+  (junction (at 140.97 96.52) (diameter 0) (color 0 0 0 0)
+  )
+  (junction (at 160.02 156.21) (diameter 0) (color 0 0 0 0)
+  )
   (junction (at 209.55 115.57) (diameter 0) (color 0 0 0 0)
   )
   (junction (at 236.22 144.78) (diameter 0) (color 0 0 0 0)
   )
+  (junction (at 143.51 93.98) (diameter 0) (color 0 0 0 0)
+  )
   (junction (at 132.08 48.26) (diameter 0) (color 0 0 0 0)
   )
@@
   (junction (at 233.68 83.82) (diameter 0) (color 0 0 0 0)
   )
+  (junction (at 165.1 151.13) (diameter 0) (color 0 0 0 0)
+  )
+  (junction (at 168.91 146.05) (diameter 0) (color 0 0 0 0)
+  )
   (junction (at 165.1 40.64) (diameter 0) (color 0 0 0 0)
   )
+  (junction (at 157.48 158.75) (diameter 0) (color 0 0 0 0)
+  )
   (junction (at 132.08 55.88) (diameter 0) (color 0 0 0 0)
   )
@@
   )
   (junction (at 209.55 144.78) (diameter 0) (color 0 0 0 0)
+  )
+  (junction (at 162.56 146.05) (diameter 0) (color 0 0 0 0)
   )
   (no_connect (at 171.45 146.05))
@@
     (stroke (width 0) (type default))
   )
-  (wire (pts (xy 168.91 143.51) (xy 168.91 163.83))
+  (wire (pts (xy 168.91 143.51) (xy 168.91 146.05))
+    (stroke (width 0) (type default))
+  )
+  (wire (pts (xy 140.97 96.52) (xy 140.97 118.11))
+    (stroke (width 0) (type default))
+  )
+  (wire (pts (xy 152.4 148.59) (xy 162.56 148.59))
     (stroke (width 0) (type default))
   )
@@
     (stroke (width 0) (type default))
   )
+  (wire (pts (xy 162.56 146.05) (xy 168.91 146.05))
+    (stroke (width 0) (type default))
+  )
   (wire (pts (xy 160.02 104.14) (xy 160.02 156.21))
     (stroke (width 0) (type default))
@@
     (stroke (width 0) (type default))
   )
-  (wire (pts (xy 121.92 93.98) (xy 170.18 93.98))
+  (wire (pts (xy 121.92 93.98) (xy 143.51 93.98))
     (stroke (width 0) (type default))
   )
@@
     (stroke (width 0) (type default))
   )
+  (wire (pts (xy 152.4 158.75) (xy 157.48 158.75))
+    (stroke (width 0) (type default))
+  )
   (wire (pts (xy 132.08 26.67) (xy 132.08 48.26))
     (stroke (width 0) (type default))
@@
     (stroke (width 0) (type default))
   )
+  (wire (pts (xy 143.51 93.98) (xy 143.51 118.11))
+    (stroke (width 0) (type default))
+  )
   (wire (pts (xy 215.9 40.64) (xy 228.6 40.64))
     (stroke (width 0) (type default))
@@
     (stroke (width 0) (type default))
   )
-  (wire (pts (xy 167.64 96.52) (xy 121.92 96.52))
+  (wire (pts (xy 167.64 96.52) (xy 140.97 96.52))
     (stroke (width 0) (type default))
   )
@@
     (stroke (width 0) (type default))
   )
+  (wire (pts (xy 135.89 115.57) (xy 135.89 118.11))
+    (stroke (width 0) (type default))
+  )
   (wire (pts (xy 167.64 107.95) (xy 167.64 96.52))
     (stroke (width 0) (type default))
   )
+  (wire (pts (xy 152.4 146.05) (xy 162.56 146.05))
+    (stroke (width 0) (type default))
+  )
+  (wire (pts (xy 168.91 146.05) (xy 168.91 163.83))
+    (stroke (width 0) (type default))
+  )
   (wire (pts (xy 121.92 73.66) (xy 218.44 73.66))
     (stroke (width 0) (type default))
@@
     (stroke (width 0) (type default))
   )
+  (wire (pts (xy 138.43 115.57) (xy 138.43 118.11))
+    (stroke (width 0) (type default))
+  )
   (wire (pts (xy 121.92 101.6) (xy 157.48 101.6))
     (stroke (width 0) (type default))
   )
+  (wire (pts (xy 165.1 153.67) (xy 165.1 151.13))
+    (stroke (width 0) (type default))
+  )
   (wire (pts (xy 121.92 55.88) (xy 132.08 55.88))
     (stroke (width 0) (type default))
@@
     (stroke (width 0) (type default))
   )
+  (wire (pts (xy 143.51 93.98) (xy 170.18 93.98))
+    (stroke (width 0) (type default))
+  )
   (wire (pts (xy 236.22 83.82) (xy 236.22 81.28))
     (stroke (width 0) (type default))
@@
     (stroke (width 0) (type default))
   )
+  (wire (pts (xy 162.56 148.59) (xy 162.56 146.05))
+    (stroke (width 0) (type default))
+  )
   (wire (pts (xy 165.1 27.94) (xy 165.1 40.64))
     (stroke (width 0) (type default))
   )
+  (wire (pts (xy 152.4 151.13) (xy 165.1 151.13))
+    (stroke (width 0) (type default))
+  )
   (wire (pts (xy 121.92 26.67) (xy 132.08 26.67))
     (stroke (width 0) (type default))
@@
     (stroke (width 0) (type default))
   )
-  (wire (pts (xy 171.45 151.13) (xy 165.1 151.13))
+  (wire (pts (xy 130.81 127) (xy 130.81 115.57))
+    (stroke (width 0) (type default))
+  )
+  (wire (pts (xy 165.1 151.13) (xy 171.45 151.13))
     (stroke (width 0) (type default))
   )
@@
     (stroke (width 0) (type default))
   )
+  (wire (pts (xy 152.4 156.21) (xy 160.02 156.21))
+    (stroke (width 0) (type default))
+  )
   (wire (pts (xy 168.91 140.97) (xy 168.91 143.51))
     (stroke (width 0) (type default))
   )
+  (wire (pts (xy 130.81 115.57) (xy 135.89 115.57))
+    (stroke (width 0) (type default))
+  )
   (wire (pts (xy 199.39 88.9) (xy 199.39 123.19))
     (stroke (width 0) (type default))
@@
     (stroke (width 0) (type default))
   )
+  (wire (pts (xy 140.97 96.52) (xy 121.92 96.52))
+    (stroke (width 0) (type default))
+  )
   (wire (pts (xy 132.08 48.26) (xy 132.08 55.88))
+    (stroke (width 0) (type default))
+  )
+  (wire (pts (xy 152.4 153.67) (xy 165.1 153.67))
     (stroke (width 0) (type default))
   )
@@
   (text "I2C (Qwiic pinout)" (at 177.8 113.03 0)
     (effects (font (size 1.27 1.27)) (justify left bottom))
+  )
+  (label "24V_PREFUSE" (at 165.1 132.08 270) (fields_autoplaced)
+    (effects (font (size 1.27 1.27)) (justify right bottom))
   )
   (symbol (lib_id "Jumper:SolderJumper_2_Bridged") (at 177.8 40.64 0) (mirror x) (unit 1)
@@
         (path "/6915e082-49b6-4d34-b3cd-1082ec18860d"
           (reference "#PWR019") (unit 1)
+        )
+      )
+    )
+  )
+  (symbol (lib_id "power:GND") (at 130.81 127 0) (unit 1)
+    (in_bom yes) (on_board yes) (dnp no) (fields_autoplaced)
+    (property "Reference" "#PWR028" (at 130.81 133.35 0)
+      (effects (font (size 1.27 1.27)) hide)
+    )
+    (property "Value" "GND" (at 130.81 132.08 0)
+      (effects (font (size 1.27 1.27)))
+    )
+    (property "Footprint" "" (at 130.81 127 0)
+      (effects (font (size 1.27 1.27)) hide)
+    )
+    (property "Datasheet" "" (at 130.81 127 0)
+      (effects (font (size 1.27 1.27)) hide)
+    )
+    (pin "1")
+    (instances
+      (project "dmxaudio"
+        (path "/6915e082-49b6-4d34-b3cd-1082ec18860d"
+          (reference "#PWR028") (unit 1)
+        )
+        (path "/6915e082-49b6-4d34-b3cd-1082ec18860d/da5620d5-8726-441a-85f6-43f0a983f61b"
+          (reference "#PWR010") (unit 1)
         )
       )
@@
       (effects (font (size 1.27 1.27)))
     )
-    (property "Footprint" "Fuse:Fuseholder_Clip-5x20mm_Keystone_3517_Inline_P23.11x6.76mm_D1.70mm_Horizontal" (at 175.26 133.858 90)
+    (property "Footprint" "dmxaudio:XF-506P" (at 175.26 133.858 90)
       (effects (font (size 1.27 1.27)) hide)
     )
@@
     )
   )
+  (symbol (lib_id "SSD1306-128x64_OLED:SSD1306") (at 139.7 127 0) (unit 1)
+    (in_bom yes) (on_board yes) (dnp no) (fields_autoplaced)
+    (property "Reference" "Brd1" (at 147.32 125.73 0)
+      (effects (font (size 1.27 1.27)) (justify left))
+    )
+    (property "Value" "SSD1306" (at 147.32 128.27 0)
+      (effects (font (size 1.27 1.27)) (justify left))
+    )
+    (property "Footprint" "dmxaudio:128x64OLED" (at 139.7 120.65 0)
+      (effects (font (size 1.27 1.27)) hide)
+    )
+    (property "Datasheet" "" (at 139.7 120.65 0)
+      (effects (font (size 1.27 1.27)) hide)
+    )
+    (pin "1")
+    (pin "2")
+    (pin "3")
+    (pin "4")
+    (instances
+      (project "dmxaudio"
+        (path "/6915e082-49b6-4d34-b3cd-1082ec18860d"
+          (reference "Brd1") (unit 1)
+        )
+      )
+    )
+  )
   (symbol (lib_id "Device:C") (at 209.55 138.43 0) (unit 1)
     (in_bom yes) (on_board yes) (dnp no) (fields_autoplaced)
@@
         (path "/6915e082-49b6-4d34-b3cd-1082ec18860d/da5620d5-8726-441a-85f6-43f0a983f61b"
           (reference "#PWR010") (unit 1)
+        )
+      )
+    )
+  )
+  (symbol (lib_id "power:+3V3") (at 138.43 115.57 0) (unit 1)
+    (in_bom yes) (on_board yes) (dnp no) (fields_autoplaced)
+    (property "Reference" "#PWR026" (at 138.43 119.38 0)
+      (effects (font (size 1.27 1.27)) hide)
+    )
+    (property "Value" "+3V3" (at 138.43 110.49 0)
+      (effects (font (size 1.27 1.27)))
+    )
+    (property "Footprint" "" (at 138.43 115.57 0)
+      (effects (font (size 1.27 1.27)) hide)
+    )
+    (property "Datasheet" "" (at 138.43 115.57 0)
+      (effects (font (size 1.27 1.27)) hide)
+    )
+    (pin "1")
+    (instances
+      (project "dmxaudio"
+        (path "/6915e082-49b6-4d34-b3cd-1082ec18860d"
+          (reference "#PWR026") (unit 1)
         )
       )
@@
         )
       )
+    )
+  )
+  (symbol (lib_id "Connector_Generic:Conn_01x06") (at 147.32 151.13 0) (mirror y) (unit 1)
+    (in_bom yes) (on_board yes) (dnp no) (fields_autoplaced)
+    (property "Reference" "J7" (at 147.32 139.7 0)
+      (effects (font (size 1.27 1.27)))
+    )
+    (property "Value" "Conn_01x06" (at 147.32 142.24 0)
+      (effects (font (size 1.27 1.27)))
+    )
+    (property "Footprint" "Connector_Molex:Molex_KK-254_AE-6410-06A_1x06_P2.54mm_Vertical" (at 147.32 151.13 0)
+      (effects (font (size 1.27 1.27)) hide)
+    )
+    (property "Datasheet" "~" (at 147.32 151.13 0)
+      (effects (font (size 1.27 1.27)) hide)
+    )
+    (pin "1")
+    (pin "2")
+    (pin "3")
+    (pin "4")
+    (pin "5")
+    (pin "6")
+    (instances
+      (project "dmxaudio"
+        (path "/6915e082-49b6-4d34-b3cd-1082ec18860d"
+          (reference "J7") (unit 1)
+        )
+      )
